File: STM32G0_MPU6050_circle.kicad_pcb (KiCad board)
At the start: 2 copper layers, 44.2 x 44.2 mm, 28 parts, among them J1 USB_B_Micro, J2 Screw_Terminal_01x02, J3 SWD_CONN_10P, Q1 Q_PMOS_GSD, U1 STM32, U2 AMS1117-3.3, U3 MPU-6050

Commit message: Setup STM32Cube
Other:
- net class Default removed

Commit message: Changed SWD pin footprint
-Changed 2x5 pin to header instead of socket. Caused orientation problems with pins on the Jtag 10-pin adapter for ST-Link debugger.
Parts:
- J3: footprint Connector_PinSocket_1.27mm:PinSocket_2x05_P1.27mm_Vertical_SMD -> Connector_PinHeader_1.27mm:PinHeader_2x05_P1.27mm_Vertical_SMD
- moved R7 2.11 mm to (172.5, 86.8)
- moved R6 2.04 mm to (173.7, 86.8)
- moved J3 0.32 mm to (175.1, 80.0), turned to -90 degrees
Routing:
- net Net-(J3-Pad4): track 2.51 -> 6.86 mm
- net Net-(J3-Pad2): track 2.52 -> 6.67 mm
- net SWDIO: track 8.20 -> 5.03 mm, vias 2 -> 0
- net SWDCLK: track 8.33 -> 6.88 mm
Other:
- board text added: "STM32G0 + MPU6050 “Walk or Run” v1.1"
- board text removed: "STM32G0 + MPU6050 “Walk or Run” v1.0"
